Commit message: update challenge 1

File: catkin_ws/src/finalproject/rotors_simulator/rotors_description/urdf/firefly.xacro (robot description, xacro)
@@ -184,63 +184,3 @@
     <xacro:insert_block name="rotor_inertia" />
   </xacro:vertical_rotor>
-<link name="connector1">
- <!--   <collision name="collision">
-      <origin xyz="0 0 0" rpy="0 0 0"/>
-      <geometry>
-      <box size="0.01 0.01 0.01"/>
-      </geometry>
-    </collision>-->
-    <visual name="connector1_visual">
-      <origin xyz="0 0 0" rpy="0 0 0"/>
-      <geometry>
-      <box size="0.01 0.01 0.01"/>
-      </geometry>
-    </visual>
-    <inertial>
-    <mass value="0.001"/>
-    <origin xyz="0.0 0 0" rpy=" 0 0 0"/>
-    <inertia
-        ixx="0.001" ixy="0" ixz="0"
-        iyy="0.001" iyz="0"
-        izz="0.001"
-    />
-    </inertial>
-  </link>
-<joint type="revolute" name="connector1_joint">
-   <origin xyz="0.0 0 -0.05" rpy="0 0 0"/>
-   <child link="connector1"/>
-   <parent link="${namespace}/base_link"/>
-   <axis xyz="0 1 0" />
-    <limit effort="300" lower="-1.57" upper="1.57" velocity="1"/>
-</joint>
-<link name="connector2">
- <!--   <collision name="collision">
-      <origin xyz="0 0 0" rpy="0 0 0"/>
-      <geometry>
-      <box size="0.01 0.01 0.01"/>
-      </geometry>
-    </collision>-->
-    <visual name="connector2_visual">
-      <origin xyz="0 0 0" rpy="0 0 0"/>
-      <geometry>
-      <box size="0.01 0.01 0.01"/>
-      </geometry>
-    </visual>
-    <inertial>
-    <mass value="0.001"/>
-    <origin xyz="0.0 0 0" rpy=" 0 0 0"/>
-    <inertia
-        ixx="0.001" ixy="0" ixz="0"
-        iyy="0.001" iyz="0"
-        izz="0.001"
-    />
-    </inertial>
-  </link>
-<joint type="revolute" name="connector2_joint">
-   <origin xyz="0.0 0 0.001" rpy="0 0 0"/>
-   <child link="connector2"/>
-   <parent link="connector1"/>
-   <axis xyz="1 0 0" />
-    <limit effort="300" lower="-1.57" upper="1.57" velocity="1"/>
-</joint>
 </robot>

File: catkin_ws/src/finalproject/rotors_simulator/rotors_description/urdf/multirotor_base.xacro (robot description, xacro)
@@ -131,17 +131,4 @@
       <material>Gazebo/${color}</material>
     </gazebo>
-<gazebo reference="${robot_namespace}/rotor_${motor_number}_joint">
-     <provideFeedback>true</provideFeedback>
-   </gazebo>
-<gazebo>
-   <plugin name="ft_sensor_2" filename="libgazebo_ros_ft_sensor.so">
-       <updateRate>100.0</updateRate>
-       <topicName>${robot_namespace}/rotor_${motor_number}_ft</topicName>
-       <jointName>${robot_namespace}/rotor_${motor_number}_joint</jointName>
-   </plugin>
-</gazebo>
-   <gazebo reference="rotor_${motor_number}">
-     <material>Gazebo/${color}</material>
-   </gazebo>
   </xacro:macro>
 </robot>
